Commit message: Added first version of DynamicsRegressorGenerator working on Python and Matlab

File: yarp/tests/test_files/icub_model.urdf (robot description, URDF)
Before this commit: robot test_icub, 55 links, 54 joints
Links:
- added link chest_skin_frame, mass 0
- link l_ankle_2: mass 0.1 -> 0.2675
- link l_foot: mass 0.761 -> 0.5935
- link r_ankle_2: mass 0.1 -> 0.2675
- link r_foot: mass 0.761 -> 0.5935
Joints:
- added joint chest_skin_frame_fixed_joint: type fixed, parent chest, child chest_skin_frame, origin xyz=0.00231 0.1933 -1.18362e-17 rpy=-1.8747e-33 5.77686e-66 6.16298e-33, axis 0 0 0
- joint codyco_balancing_world_fixed_joint: origin xyz=-8.67362e-19 -1.38778e-17 0.075 rpy=3.14159 -0 0 -> xyz=-8.67362e-19 -1.38778e-17 0.004 rpy=3.14159 -0 0
- joint l_foot_dh_frame_fixed_joint: origin xyz=-8.67362e-19 -1.38778e-17 0.075 rpy=-9.70754e-18 1.5708 -9.70754e-18 -> xyz=0 0 0.004 rpy=0 1.5708 0
- joint l_foot_ft_sensor: origin xyz=-0.0035 0 -0.0065 rpy=0 -0 0 -> xyz=-0.0035 0 0.0645 rpy=0 -0 0
- joint l_sole_fixed_joint: origin xyz=0 0 0.075 rpy=0 1.5708 0 -> xyz=-8.67362e-19 -1.38778e-17 0.004 rpy=3.14159 -0 0
- joint r_foot_dh_frame_fixed_joint: origin xyz=-4.29004e-17 -0.1362 0.075 rpy=-0.834365 1.5708 -0.834365 -> xyz=0 0 0.004 rpy=0 1.5708 0
- joint r_foot_ft_sensor: origin xyz=-0.0035 4.28626e-19 -0.0065 rpy=0 -0 0 -> xyz=-0.0035 4.28626e-19 0.0645 rpy=0 -0 0
- joint r_sole_fixed_joint: origin xyz=0 0 0.075 rpy=0 1.5708 0 -> xyz=-8.67362e-19 1.38778e-17 0.004 rpy=3.14159 -0 0
