Commit message: Bug fix in conversion between iDynTree and KDL free floating state, account for different serializations

File: tests/data/icubTwoLinks.urdf (robot description, URDF)
Before this commit: robot test_icub, 3 links, 2 joints
Links:
- removed link torso_1
- added link l_hip_1, mass 0.754; collision mesh filename=meshes/collision/icub_simple_collision_l_hip_1.dae scale=1 1 1; visual mesh filename=meshes/visual/icub_l_hip_1.dae scale=1 1 1
Joints:
- removed joint torso_pitch
- added joint l_hip_pitch: type revolute, parent root_link, child l_hip_1, origin xyz=0 -0.0681 -0.1199 rpy=-3.14159 1.5708 -2.77556e-17, axis 0 -1 6.12323e-17, limit lower=-0.767945 upper=2.30383 effort=84 velocity=100

File: tests/data/twoLinks.urdf (robot description, URDF)
Before this commit: robot twoLinks, 3 links, 2 joints
Joints:
- joint joint_1_2: origin xyz=0 0 0 rpy=0 -0 0 -> xyz=1 0 0 rpy=0 -0 0
