Commit message: Added handling of collision and visual shapes in reduce model functions
Furtheremore, add first test of visualization, to check that a reduced
model is correctly visualized. For now the tests require a graphical enviroment.

File: src/tests/data/threeLinks.urdf (robot description, URDF)
Before this commit: robot twoLinks, 4 links, 3 joints
Links:
- link link1: geometry collision box size=1 1 1; visual box size=1 1 1
- link link2: geometry collision box size=1 1 1; visual box size=1 1 1
- link link3: geometry collision box size=1 1 1; visual box size=1 1 1
