Commit message: Added first model tranformer function: removeFakeLinks
This function is used in the URDF parser to remove
"fake links" and transform them in "frames"

Added some frames as "fake links" to the oneLink.urdf
test model , to test the behaviour of this new function in
URDFModelImportUnitTest .

File: src/tests/data/oneLink.urdf (robot description, URDF)
Before this commit: robot oneLink, 2 links, 1 joints
Links:
- added link frame1, mass 0.0
- added link frame2, mass 0.0
Joints:
- added joint frame1_fixed_joint: type fixed, parent link1, child frame1, origin xyz=0 10 0 rpy=0 -30 0, axis 0 0 0
- added joint frame2_fixed_joint: type fixed, parent link1, child frame2, origin xyz=0 30 0 rpy=0 0.0 0, axis 0 0 0

Commit message: Fix malformed oneLinks.urdf that was causing a failure in the tests

File: src/tests/data/oneLink.urdf (robot description, URDF)
Before this commit: robot oneLink, 4 links, 3 joints
Joints:
- joint frame2_fixed_joint: origin xyz=0 30 0 rpy=0 0.0 0 -> xyz=0 30 0 rpy=0.0 0.0 0.0

Commit message: Add support for handling scale in InertialParametersSolidShapesHelpers
Originally contributed in https://github.com/robotology/idyntree/pull/577/files

File: src/tests/data/oneLink.urdf (robot description, URDF)
Before this commit: robot oneLink, 4 links, 3 joints
Links:
- link link1: geometry collision mesh filename=cube.stl scale=0.1 0.1 0.1; visual mesh filename=cube.stl scale=0.1 0.1 0.1
